File: hackday13.kicad_pcb (KiCad board)
At the start: 4 copper layers, 100 x 100 mm, 40 parts, among them J1 TT-output, J2 TT-input, J3 TT-bidirectional, J4 Conn_01x02_Pin, J5 Conn_01x02_Pin, J6 Conn_01x02_Pin, J7 Conn_01x02_Pin, SW1 Reset button, SW2 SW_DIP_x02, U1 MCP73831-4-OT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

Commit message: Add initial placement
Parts:
- removed BT2: Battery_Cell, Battery:BatteryHolder_Keystone_3002_1x2032
- removed ShReg1, ShReg2: MC14014B, Package_SO:SOIC-16_3.9x9.9mm_P1.27mm
- removed ShReg3: 74HC595, Package_SO:SOIC-16_3.9x9.9mm_P1.27mm
- added BT1: Battery_Cell, Battery:BatteryHolder_Keystone_3002_1x2032, F.Cu at (94.2, 116.0)
- added D6: LED, LED_THT:LED_D3.0mm, F.Cu at (160.0, 48.0)
- added D7: LED, LED_THT:LED_D3.0mm, F.Cu at (76.5, 63.5)
- added R14: 0, Resistor_THT:R_Axial_DIN0207_L6.3mm_D2.5mm_P10.16mm_Horizontal, F.Cu at (82.0, 69.0)
- added R15: 0, Resistor_THT:R_Axial_DIN0207_L6.3mm_D2.5mm_P10.16mm_Horizontal, F.Cu at (82.3, 73.5)
- added R16: 0, Resistor_THT:R_Axial_DIN0207_L6.3mm_D2.5mm_P10.16mm_Horizontal, F.Cu at (128.9, 52.0)
- added R17: 0, Resistor_THT:R_Axial_DIN0207_L6.3mm_D2.5mm_P10.16mm_Horizontal, F.Cu at (142.8, 52.0)
- added R18: 200 Ohm, Resistor_THT:R_Axial_DIN0207_L6.3mm_D2.5mm_P10.16mm_Horizontal, F.Cu at (160.5, 43.0)
- added R19: 200 Ohm, Resistor_THT:R_Axial_DIN0207_L6.3mm_D2.5mm_P10.16mm_Horizontal, F.Cu at (81.8, 61.0)
- added U3: 74HC165, Package_DIP:DIP-16_W7.62mm, F.Cu at (129.5, 41.0)
- added U4: 74HC165, Package_DIP:DIP-16_W7.62mm, F.Cu at (155.5, 41.0)
- added U5: 74HC595, Package_DIP:DIP-16_W7.62mm, F.Cu at (103.5, 41.0)
- R13: value 1000 Ohm -> 200 Ohm
- moved D1 179.0 mm to (81.2, 91.5)
- moved D5 178.7 mm to (77.0, 73.0)
- moved D4 177.3 mm to (81.2, 96.0)
- moved J7 173.2 mm to (78.0, 54.5)
- moved D3 169.3 mm to (88.8, 101.0), turned to 180 degrees
- moved SW1 149.5 mm to (98.5, 92.5), turned to 90 degrees
- moved TP3 146.8 mm to (80.0, 85.0)
- moved C2 142.7 mm to (116.5, 105.0), turned to -90 degrees
- moved U1 139.8 mm to (119.9, 99.5)
- moved D2 139.7 mm to (112.8, 94.0), turned to 180 degrees
- moved C1 137.1 mm to (126.0, 119.5), turned to -90 degrees
- moved J5 133.8 mm to (115.0, 120.5)
- moved R13 129.8 mm to (79.4, 78.5)
- moved TP1 129.6 mm to (97.5, 99.5)
- moved R11 129.4 mm to (81.9, 56.5)
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Connections:
- D5 pad 1: GND -> Net-(D5-K)
- D5 pad 2: Net-(D5-A) -> +3.3V
- R1 pad 2: Net-(U2-GPIO12) -> Net-(U2-GPIO0)
- R11 pad 1: VCC -> +3.3V
- R13 pad 1: Net-(D5-A) -> Net-(D5-K)
- R2 pad 2: Net-(U2-GPIO13) -> Net-(U2-GPIO1)
- R3 pad 2: Net-(U2-GPIO14) -> Net-(U2-GPIO2)
- R4 pad 2: Net-(U2-GPIO15) -> Net-(U2-GPIO3)
- U2 pad 1: Net-(ShReg3-RCLK) -> Net-(U2-GPIO0)
- U2 pad 11: Net-(ShReg1-P/S) -> /CLK
- U2 pad 12: Net-(J4-Pin_1) -> /SH/NLD
- U2 pad 14: Net-(J4-Pin_2) -> Net-(U2-GPIO10)
- U2 pad 15: /charge_ind -> /CLK
- U2 pad 16: Net-(U2-GPIO12) -> /SH/NLD
- U2 pad 17: Net-(U2-GPIO13) -> Net-(J4-Pin_1)
- U2 pad 19: Net-(U2-GPIO14) -> Net-(J4-Pin_2)
- U2 pad 2: Net-(ShReg3-SRCLK) -> Net-(U2-GPIO1)
- U2 pad 20: Net-(U2-GPIO15) -> /charge_ind
- U2 pad 4: Net-(ShReg3-SER) -> Net-(U2-GPIO2)
- U2 pad 5: Net-(ShReg2-Q8) -> Net-(U2-GPIO3)
