File: hackday13.kicad_pcb (KiCad board)
At the start: 4 copper layers, 100 x 100 mm, 40 parts, among them J1 TT-output, J2 TT-input, J3 TT-bidirectional, J4 Conn_01x02_Pin, J5 Conn_01x02_Pin, J6 Conn_01x02_Pin, J7 Conn_01x02_Pin, SW1 Reset button, SW2 SW_DIP_x02, U1 MCP73831-4-OT, U2 RaspberryPi_Pico_W

Commit message: [layout] first version of possible layout - review required
Parts:
- removed J4: Conn_01x02_Pin, Connector_PinHeader_2.54mm:PinHeader_1x02_P2.54mm_Vertical
- removed ShReg1, ShReg2: MC14014B, Package_SO:SOIC-16_3.9x9.9mm_P1.27mm
- removed ShReg3: 74HC595, Package_SO:SOIC-16_3.9x9.9mm_P1.27mm
- added C3: 100n, Capacitor_THT:C_Disc_D7.0mm_W2.5mm_P5.00mm, F.Cu at (113.8, 59.1)
- added C4: 100n, Capacitor_THT:C_Disc_D7.0mm_W2.5mm_P5.00mm, F.Cu at (136.9, 58.9)
- added C5: 100n, Capacitor_THT:C_Disc_D7.0mm_W2.5mm_P5.00mm, F.Cu at (104.1, 42.5)
- added D6: LED, LED_THT:LED_D3.0mm, F.Cu at (152.4, 43.7)
- added G***: LOGO, custom_components_led_pcb:logo, F.Cu at (127.6, 110.8)
- added H1: MountingHole, MountingHole:MountingHole_3.2mm_M3, F.Cu at (157.0, 37.6)
- added H2: MountingHole, MountingHole:MountingHole_3.2mm_M3, F.Cu at (111.0, 47.5)
- added H3: MountingHole, MountingHole:MountingHole_3.2mm_M3, F.Cu at (139.4, 125.7)
- added H4: MountingHole, MountingHole:MountingHole_3.2mm_M3, F.Cu at (90.9, 122.7)
- added J8: Conn_01x03_Pin, Connector_PinHeader_2.54mm:PinHeader_1x03_P2.54mm_Vertical, F.Cu at (121.4, 92.5)
- added R14: 0, Resistor_SMD:R_0805_2012Metric, F.Cu at (114.0, 41.1)
- added R15: 0, Resistor_SMD:R_0805_2012Metric, F.Cu at (136.8, 43.7)
- added R16: 2.2k Ohm, Resistor_THT:R_Axial_DIN0207_L6.3mm_D2.5mm_P10.16mm_Horizontal, F.Cu at (152.4, 48.8)
- added U3: 74HC595, Package_DIP:DIP-16_W7.62mm, F.Cu at (93.5, 42.4)
- added U4: 74HC165, Package_DIP:DIP-16_W7.62mm, F.Cu at (124.7, 59.2)
- added U5: 74HC165, Package_DIP:DIP-16_W7.62mm, F.Cu at (147.6, 58.9)
- BT2: moved to B.Cu
- R11: footprint Resistor_THT:R_Axial_DIN0207_L6.3mm_D2.5mm_P10.16mm_Horizontal -> Resistor_SMD:R_0805_2012Metric
- R12: value 0 -> 2.2k Ohm
- R13: value 1000 Ohm -> 0; footprint Resistor_THT:R_Axial_DIN0207_L6.3mm_D2.5mm_P10.16mm_Horizontal -> Resistor_SMD:R_0805_2012Metric
- moved D4 168.8 mm to (89.4, 100.3), turned to -90 degrees
- moved C2 159.4 mm to (100.6, 111.5), turned to 90 degrees
- moved D1 154.8 mm to (109.0, 62.7), turned to 90 degrees
- moved U1 154.0 mm to (105.0, 109.0)
- moved C1 153.6 mm to (107.4, 112.8), turned to -90 degrees
- moved J6 146.6 mm to (95.5, 108.0), turned to -90 degrees
- moved J5 145.3 mm to (104.1, 124.2), turned to -90 degrees
- moved D2 143.7 mm to (108.7, 96.3)
- moved D3 141.1 mm to (117.3, 94.5), turned to -90 degrees
- moved D5 138.1 mm to (129.6, 43.9), turned to -90 degrees
- moved TP1 136.2 mm to (90.7, 93.2)
- moved TP3 127.6 mm to (98.0, 94.7)
- moved R6 119.1 mm to (96.0, 101.6)
- moved R13 112.1 mm to (104.3, 50.0), turned to 180 degrees
- moved R11 107.3 mm to (104.3, 57.7), turned to 180 degrees
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Connections:
- D5 pad 1: GND -> Net-(D5-K)
- J1 pad 1: Net-(J1-IO1) -> /OUT_1
- J1 pad 10: Net-(J1-IO8) -> /OUT_8
- J1 pad 2: Net-(J1-IO2) -> /OUT_2
- J1 pad 3: Net-(J1-IO3) -> /OUT_3
- J1 pad 4: Net-(J1-IO4) -> /OUT_4
- J1 pad 7: Net-(J1-IO5) -> /OUT_5
- J1 pad 8: Net-(J1-IO6) -> /OUT_6
- J1 pad 9: Net-(J1-IO7) -> /OUT_7
- J2 pad 1: Net-(J2-IO1) -> /IN1
- J2 pad 10: Net-(J2-IO8) -> /IN8
- J2 pad 2: Net-(J2-IO2) -> /IN2
- J2 pad 3: Net-(J2-IO3) -> /IN3
- J2 pad 4: Net-(J2-IO4) -> /IN4
- J2 pad 7: Net-(J2-IO5) -> /IN5
- J2 pad 8: Net-(J2-IO6) -> /IN6
- J2 pad 9: Net-(J2-IO7) -> /IN7
- J3 pad 1: Net-(J3-IO1) -> /INOUT_1
- J3 pad 10: Net-(J3-IO8) -> /INOUT_8
- J3 pad 2: Net-(J3-IO2) -> /INOUT_2
- J3 pad 3: Net-(J3-IO3) -> /INOUT_3
- J3 pad 4: Net-(J3-IO4) -> /INOUT_4
- J3 pad 7: Net-(J3-IO5) -> /INOUT_5
- J3 pad 8: Net-(J3-IO6) -> /INOUT_6
- J3 pad 9: Net-(J3-IO7) -> /INOUT_7
- R1 pad 2: Net-(U2-GPIO12) -> /DotMat_C1
- R10 pad 2: Net-(U2-GPIO27_ADC1) -> Net-(U2-GPIO16)
- R12 pad 1: GND -> Net-(D5-A)
- R12 pad 2: Net-(ShReg3-~{OE}) -> VCC
- R13 pad 1: Net-(D5-A) -> GND
- R2 pad 2: Net-(U2-GPIO13) -> /DotMat_C5
- R3 pad 2: Net-(U2-GPIO14) -> /DotMat_C2
- R4 pad 2: Net-(U2-GPIO15) -> /DotMat_C4
- R5 pad 2: Net-(U2-GPIO16) -> /DotMat_C3
- R9 pad 2: Net-(U2-GPIO28_ADC2) -> Net-(U2-GPIO17)
- SW2 pad 3: Net-(U2-GPIO27_ADC1) -> Net-(U2-GPIO16)
- SW2 pad 4: Net-(U2-GPIO28_ADC2) -> Net-(U2-GPIO17)
- U2 pad 10: Net-(ShReg1-Clk) -> /OPS
- U2 pad 16: Net-(U2-GPIO12) -> /DotMat_C5
- U2 pad 17: Net-(U2-GPIO13) -> /DotMat_C4
- U2 pad 19: Net-(U2-GPIO14) -> /DotMat_C3
- U2 pad 20: Net-(U2-GPIO15) -> /DotMat_C2
- U2 pad 22: /DotMat_R1 -> Net-(U2-GPIO17)
- U2 pad 24: /DotMat_R2 -> /DotMat_R1
- U2 pad 25: /DotMat_R3 -> /DotMat_R2
- U2 pad 26: /DotMat_R4 -> /DotMat_C1
- U2 pad 27: /DotMat_R5 -> /DotMat_R4
- U2 pad 29: /DotMat_R6 -> /DotMat_R3
- U2 pad 31: /DotMat_R7 -> /DotMat_R5
- U2 pad 32: Net-(U2-GPIO27_ADC1) -> /DotMat_R6
- U2 pad 34: Net-(U2-GPIO28_ADC2) -> /DotMat_R7
- U2 pad 5: Net-(ShReg2-Q8) -> /Set_Data_1
- U2 pad 6: Net-(ShReg2-Clk) -> /Set_Data_2
- U2 pad 7: Net-(ShReg2-P/S) -> /CLK_EN
- U2 pad 9: Net-(ShReg1-Q8) -> /CLK
Routing:
- net +3.3V: track 0.00 -> 131.0 mm, vias 0 -> 1
- net /DotMat_R7: track 0.00 -> 83.0 mm
- net /DotMat_R6: track 0.00 -> 77.4 mm
- net /Set_Data_2: track 0.00 -> 76.0 mm
- net /CLK_EN: track 0.00 -> 73.5 mm
- net /DotMat_R5: track 0.00 -> 72.4 mm
- net /DotMat_R4: track 0.00 -> 70.0 mm
- net /CLK: track 0.00 -> 69.5 mm
- net /DotMat_R2: track 0.00 -> 66.5 mm, vias 0 -> 1
- net /DotMat_R3: track 0.00 -> 65.1 mm
- net /DotMat_R1: track 0.00 -> 64.6 mm, vias 0 -> 1
- net /OPS: track 0.00 -> 63.9 mm
- net /Set_Data_1: track 0.00 -> 55.9 mm
- net Net-(U2-RUN): track 0.00 -> 53.2 mm
- net /charge_ind: track 0.00 -> 49.0 mm
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- added copper zone on F.Cu, net +5V
- added copper zone on In1.Cu, net +5V
- added copper zone on In1.Cu, net +BATT
- added copper zone on F.Cu, net /Bat_Chg
- added copper zone on B.Cu, net GND
- added copper zone on F.Cu, net GND
- added copper zone on In1.Cu, net GND
- added copper zone on In1.Cu, net Net-(BT2-+)
- added copper zone on In1.Cu, net VCC
Other:
- board size 100 x 100 mm -> 76.6 x 100 mm
- board text added: "100n"
- board text added: "3.3V"
- board text added: "4.7u"
- board text added: "5V"
- board text added: "74HC165"
- board text added: "74HC595"
- board text added: "Bat"
- board text added: "BiDir"
- board text added: "Charge"
- board text added: "Copper"
- board text added: "DBG SW"
- board text added: "Exposed"
- board text added: "Exposed Copper Keep Out"
- board text added: "Hackday 19"
- board text added: "In"
- board text added: "Keep"
- board text added: "Keep Out"
- board text added: "Marno Ray Raphael"
- board text added: "Out"
- board text added: "RST"
- board text added: "Serial Data"
- board text added: "VCC"
- board text added: "spare"
