File: hackday13.kicad_sch (KiCad schematic)
At the start: 48 parts, among them J1 TT-output, J2 TT-input, J3 TT-bidirectional, J4 Conn_01x02_Pin, J5 Conn_01x02_Pin, J6 Conn_01x02_Pin, J7 Conn_01x02_Pin, SW1 Reset button, SW2 SW_DIP_x02, U1 MCP73831-4-OT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

Commit message: Hackday 19 added to title
Other:
- title: Hackday 13 & 14 -> Hackday 13 & 14 & 19
Changed lines of the file:
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@@
 	(paper "A4")
 	(title_block
-		(title "Hackday 13 & 14")
+		(title "Hackday 13 & 14 & 19")
 		(date "2024-03-15")
 		(rev "0")
